File: DistanceSensors&IMU.kicad_sch (KiCad schematic)
At the start: 0 parts

Commit message: cos tam cos tam
Parts:
- added D401, D402, D403, D404, D405, D406: LED, symbol Device:LED
- added IC401: ULN2003ADR, SOIC127P600X175-16N, symbol SamacSys_Parts:ULN2003ADR
- added Q401, Q402, Q403, Q404, Q405, Q406: Q_Photo_NPN, symbol Device:Q_Photo_NPN
- added R208 (x6): 22, symbol Device:R_Small
- added R208 (x6): 1k, symbol Device:R_Small
Connections:
- new net: D402.1 (K), IC401.12 (5C)
- new net: D402.2 (A), R208.2
- new net: D401.2 (A), R208.2
- new net: D406.2 (A), R208.2
- new net: D403.2 (A), R208.2
- new net: D401.1 (K), IC401.11 (6C)
- new net: D403.1 (K), IC401.13 (4C)
- new net: D404.1 (K), IC401.14 (3C)
- new net: D405.1 (K), IC401.15 (2C)
- new net: D406.1 (K), IC401.16 (1C)
- new net: D405.2 (A), R208.2
- new net: D404.2 (A), R208.2
- new net +5V: Q401.1 (C), Q402.1 (C), Q403.1 (C), Q404.1 (C), Q405.1 (C), Q406.1 (C), R208.1, R208.1, R208.1, R208.1, R208.1, R208.1
- new net GND: IC401.8 (E), R208.1, R208.1, R208.1, R208.1, R208.1, R208.1
- new net IR_1: IC401.1 (1B)
- new net IR_2: IC401.2 (2B)
- new net IR_3: IC401.3 (3B)
- new net IR_4: IC401.4 (4B)
- new net IR_5: IC401.5 (5B)
- new net IR_6: IC401.6 (6B)
- new net REC_1: Q401.2 (E), R208.2
- new net REC_2: Q402.2 (E), R208.2
- new net REC_3: Q403.2 (E), R208.2
- new net REC_4: Q404.2 (E), R208.2
- new net REC_5: Q405.2 (E), R208.2
- new net REC_6: Q406.2 (E), R208.2
- no-connect marks 0 -> 3
Other:
- note added: "Diode max dc current = 100mA"
- note added: "IR & Photo placed in one led case"
- note added: "Id = 3.5V/22Ohm = 0.16A"
- note added: "Power diodes only by PWM < 60%"
- note added: "[2] IR RECEIVERS & TRANSMITERS"
