File: Micromouse.kicad_sch (KiCad schematic)
At the start: 0 parts

Commit message: working...
Other:
- sheet Distance_sensors_&_IMU renamed Distance_sensors
- sheet Distance_sensors: file DistanceSensors&IMU.kicad_sch -> DistanceSensors.kicad_sch
- note removed: "ACC & GYRO BMI088"
Changed lines of the file:
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@@
-    (effects (font (size 1.27 1.27) (thickness 0.254) bold) (justify left bottom))
-  )
-  (text "ACC & GYRO BMI088 " (at 71.628 92.202 0)
     (effects (font (size 1.27 1.27) (thickness 0.254) bold) (justify left bottom))
   )
@@
     (stroke (width 0.1524) (type solid))
     (fill (color 0 0 0 0.0000))
-    (property "Sheetname" "Distance_sensors_&_IMU" (at 69.85 81.3304 0)
+    (property "Sheetname" "Distance_sensors" (at 69.85 81.3304 0)
       (effects (font (size 1.27 1.27)) (justify left bottom))
     )
-    (property "Sheetfile" "DistanceSensors&IMU.kicad_sch" (at 69.85 108.5346 0)
+    (property "Sheetfile" "DistanceSensors.kicad_sch" (at 69.85 108.5346 0)
       (effects (font (size 1.27 1.27)) (justify left top))
     )

Commit message: Prawie skończone
Other:
- removed sheet Wireless_communication 
- added sheet IMU (imu.kicad_sch)
- note removed: "HC-05 or ESP32 (?)"
Changed lines of the file:
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@@
 (kicad_sch (version 20230121) (generator eeschema)
   (paper "A4")
-  (polyline (pts (xy 110.744 63.754) (xy 110.744 127.762))
+  (polyline (pts (xy 109.22 65.532) (xy 109.22 129.54))
     (stroke (width 0.5) (type default) (color 255 0 47 1))
   )
@@
     (stroke (width 0.5) (type default) (color 255 0 47 1))
   )
-  (polyline (pts (xy 127.508 63.754) (xy 110.744 63.754))
+  (polyline (pts (xy 127.508 65.532) (xy 109.22 65.532))
     (stroke (width 0.5) (type default) (color 255 0 47 1))
   )
@@
     (effects (font (size 2 2) (thickness 0.254) bold) (justify left bottom))
   )
-  (text "[1] Micromouse - Top level Schematic" (at 19.304 21.844 0)
+  (text "[1] Micromouse - Top level Schematic" (at 20.32 22.86 0)
     (effects (font (size 5 5) (thickness 1) bold) (justify left bottom))
   )
   (text "Hierarchical Sheet" (at 183.642 175.641 0)
     (effects (font (size 3 3) (thickness 0.6) bold) (justify left bottom))
-  )
-  (text "HC-05 or ESP32 (?) " (at 81.788 137.922 0)
-    (effects (font (size 1.27 1.27) (thickness 0.254) bold) (justify left bottom))
   )
   (text "BATTERY: LI-PO 2S,\nCONVERTERS: BUCK, LDO" (at 139.954 60.96 0)
@@
   (text "IR DIODE & FOTOTRANSISTORS" (at 71.374 88.392 0)
     (effects (font (size 1.27 1.27) (thickness 0.254) bold) (justify left bottom))
-  )
-  (sheet (at 74.168 127.762) (size 37.084 21.082) (fields_autoplaced)
-    (stroke (width 0.1524) (type solid))
-    (fill (color 0 0 0 0.0000))
-    (property "Sheetname" "Wireless_communication " (at 74.168 127.0504 0)
-      (effects (font (size 1.27 1.27)) (justify left bottom))
-    )
-    (property "Sheetfile" "WirelssCOM.kicad_sch" (at 74.168 149.4286 0)
-      (effects (font (size 1.27 1.27)) (justify left top))
-    )
-    (instances
-      (project "Micromouse"
-        (path "/4e1363f1-0338-4205-b4c3-be947d5bb41d" (page "5"))
-      )
-    )
   )
   (sheet (at 189.738 81.407) (size 44.45 25.781) (fields_autoplaced)
@@
     (instances
       (project "Micromouse"
-        (path "/4e1363f1-0338-4205-b4c3-be947d5bb41d" (page "3"))
+        (path "/4e1363f1-0338-4205-b4c3-be947d5bb41d" (page "4"))
       )
     )
@@
     )
     (property "Sheetfile" "Power.kicad_sch" (at 127.508 69.9266 0)
+      (effects (font (size 1.27 1.27)) (justify left top))
+    )
+    (instances
+      (project "Micromouse"
+        (path "/4e1363f1-0338-4205-b4c3-be947d5bb41d" (page "2"))
+      )
+    )
+  )
+  (sheet (at 86.36 129.54) (size 35.56 17.78) (fields_autoplaced)
+    (stroke (width 0.1524) (type solid))
+    (fill (color 0 0 0 0.0000))
+    (property "Sheetname" "IMU" (at 86.36 128.8284 0)
+      (effects (font (size 1.27 1.27)) (justify left bottom))
+    )
+    (property "Sheetfile" "imu.kicad_sch" (at 86.36 147.9046 0)
       (effects (font (size 1.27 1.27)) (justify left top))
     )
@@
     (instances
       (project "Micromouse"
-        (path "/4e1363f1-0338-4205-b4c3-be947d5bb41d" (page "4"))
+        (path "/4e1363f1-0338-4205-b4c3-be947d5bb41d" (page "5"))
       )
     )
@@
     (instances
       (project "Micromouse"
-        (path "/4e1363f1-0338-4205-b4c3-be947d5bb41d" (page "2"))
+        (path "/4e1363f1-0338-4205-b4c3-be947d5bb41d" (page "3"))
       )
     )

Commit message: Dodaje wszystko nie chce mi sie z tym bawic
Other:
- note added: "ACC & GYRO"
- note added: "BATTERY: LI-PO 2S, CONVERTERS: LDO"
- note removed: "BATTERY: LI-PO 2S, CONVERTERS: BUCK, LDO"
Changed lines of the file:
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@@
 (kicad_sch (version 20230121) (generator eeschema)
   (paper "A4")
-  (polyline (pts (xy 109.22 65.532) (xy 109.22 129.54))
-    (stroke (width 0.5) (type default) (color 255 0 47 1))
+  (junction (at 96.52 66.04) (diameter 0) (color 255 4 15 1)
   )
-  (polyline (pts (xy 127.508 58.42) (xy 102.87 58.42))
-    (stroke (width 0.5) (type default) (color 255 0 47 1))
+  (junction (at 96.52 48.26) (diameter 0) (color 255 4 15 1)
   )
-  (polyline (pts (xy 127.508 65.532) (xy 109.22 65.532))
-    (stroke (width 0.5) (type default) (color 255 0 47 1))
+  (junction (at 96.52 78.74) (diameter 0) (color 255 4 15 1)
   )
-  (polyline (pts (xy 156.972 69.342) (xy 156.972 82.042))
-    (stroke (width 0.5) (type default) (color 255 0 47 1))
+  (wire (pts (xy 162.56 48.26) (xy 167.64 48.26))
+    (stroke (width 0.5) (type default) (color 255 10 12 1))
   )
-  (polyline (pts (xy 206.248 59.944) (xy 206.248 81.28))
-    (stroke (width 0.5) (type default) (color 255 0 47 1))
+  (wire (pts (xy 96.52 48.26) (xy 106.68 48.26))
+    (stroke (width 0.5) (type default) (color 255 4 15 1))
   )
-  (polyline (pts (xy 102.87 58.42) (xy 102.87 81.788))
-    (stroke (width 0.5) (type default) (color 255 0 47 1))
+  (wire (pts (xy 76.2 71.12) (xy 76.2 48.26))
+    (stroke (width 0.5) (type default) (color 255 4 15 1))
   )
-  (polyline (pts (xy 183.642 59.944) (xy 206.248 59.944))
-    (stroke (width 0.5) (type default) (color 255 0 47 1))
+  (wire (pts (xy 71.12 71.12) (xy 71.12 43.18))
+    (stroke (width 0.5) (type default) (color 255 17 1 1))
   )
-  (text "DC engines & Motor driver & Encoders\n" (at 191.262 92.964 0)
+  (wire (pts (xy 96.52 66.04) (xy 96.52 48.26))
+    (stroke (width 0.5) (type default) (color 255 4 15 1))
+  )
+  (wire (pts (xy 167.64 48.26) (xy 167.64 73.66))
+    (stroke (width 0.5) (type default) (color 255 10 12 1))
+  )
+  (wire (pts (xy 76.2 48.26) (xy 96.52 48.26))
+    (stroke (width 0.5) (type default) (color 255 4 15 1))
+  )
+  (wire (pts (xy 157.48 76.2) (xy 157.48 66.04))
+    (stroke (width 0.5) (type default) (color 255 10 12 1))
+  )
+  (wire (pts (xy 167.64 73.66) (xy 170.18 73.66))
+    (stroke (width 0.5) (type default) (color 255 10 12 1))
+  )
+  (wire (pts (xy 71.12 43.18) (xy 106.68 43.18))
+    (stroke (width 0.5) (type default) (color 255 17 1 1))
+  )
+  (wire (pts (xy 157.48 66.04) (xy 96.52 66.04))
+    (stroke (width 0.5) (type default) (color 255 4 15 1))
+  )
+  (wire (pts (xy 114.3 78.74) (xy 96.52 78.74))
+    (stroke (width 0.5) (type default) (color 255 4 15 1))
+  )
+  (wire (pts (xy 170.18 76.2) (xy 157.48 76.2))
+    (stroke (width 0.5) (type default) (color 255 10 12 1))
+  )
+  (wire (pts (xy 96.52 78.74) (xy 96.52 66.04))
+    (stroke (width 0.5) (type default) (color 255 4 15 1))
+  )
+  (wire (pts (xy 96.52 119.38) (xy 96.52 78.74))
+    (stroke (width 0.5) (type default) (color 255 4 15 1))
+  )
+  (text "DC engines & Motor driver & Encoders\n" (at 170.942 82.804 0)
     (effects (font (size 1.27 1.27) (thickness 0.254) bold) (justify left bottom))
   )
-  (text "STM32F405RGT6" (at 138.176 109.22 0)
+  (text "ACC & GYRO" (at 76.2 129.54 0)
+    (effects (font (size 1.27 1.27) (thickness 0.254) bold) (justify left bottom))
+  )
+  (text "STM32F405RGT6" (at 117.856 99.06 0)
     (effects (font (size 2 2) (thickness 0.254) bold) (justify left bottom))
   )
@@
     (effects (font (size 3 3) (thickness 0.6) bold) (justify left bottom))
   )
-  (text "BATTERY: LI-PO 2S,\nCONVERTERS: BUCK, LDO" (at 139.954 60.96 0)
+  (text "BATTERY: LI-PO 2S,\nCONVERTERS: LDO" (at 119.634 50.8 0)
     (effects (font (size 1.27 1.27) (thickness 0.254) bold) (justify left bottom))
   )
-  (text "IR DIODE & FOTOTRANSISTORS" (at 71.374 88.392 0)
+  (text "IR DIODE & FOTOTRANSISTORS" (at 52.7244 82.2634 0)
     (effects (font (size 1.27 1.27) (thickness 0.254) bold) (justify left bottom))
   )
-  (sheet (at 189.738 81.407) (size 44.45 25.781) (fields_autoplaced)
+  (hierarchical_label "3V3" (shape input) (at 114.3 78.74 0) (fields_autoplaced)
+    (effects (font (size 1.27 1.27)) (justify left))
+  )
+  (hierarchical_label "3V3" (shape input) (at 76.2 71.12 270) (fields_autoplaced)
+    (effects (font (size 1.27 1.27)) (justify right))
+  )
+  (hierarchical_label "VBatt" (shape input) (at 162.56 48.26 180) (fields_autoplaced)
+    (effects (font (size 1.27 1.27)) (justify right))
+  )
+  (hierarchical_label "5V" (shape input) (at 106.68 43.18 0) (fields_autoplaced)
+    (effects (font (size 1.27 1.27)) (justify left))
+  )
+  (hierarchical_label "3V3" (shape input) (at 96.52 119.38 270) (fields_autoplaced)
+    (effects (font (size 1.27 1.27)) (justify right))
+  )
+  (hierarchical_label "3V3" (shape input) (at 106.68 48.26 0) (fields_autoplaced)
+    (effects (font (size 1.27 1.27)) (justify left))
+  )
+  (hierarchical_label "VBatt" (shape input) (at 170.18 73.66 0) (fields_autoplaced)
+    (effects (font (size 1.27 1.27)) (justify left))
+  )
+  (hierarchical_label "5V" (shape input) (at 71.12 71.12 270) (fields_autoplaced)
+    (effects (font (size 1.27 1.27)) (justify right))
+  )
+  (hierarchical_label "3V3" (shape input) (at 170.18 76.2 0) (fields_autoplaced)
+    (effects (font (size 1.27 1.27)) (justify left))
+  )
+  (sheet (at 170.18 71.12) (size 43.18 25.4) (fields_autoplaced)
     (stroke (width 0.1524) (type solid))
     (fill (color 0 0 0 0.0000))
-    (property "Sheetname" "Motors" (at 189.738 80.6954 0)
+    (property "Sheetname" "Motors" (at 170.18 70.4084 0)
       (effects (font (size 1.27 1.27)) (justify left bottom))
     )
-    (property "Sheetfile" "Motors.kicad_sch" (at 189.738 107.7726 0)
+    (property "Sheetfile" "Motors.kicad_sch" (at 170.18 97.4856 0)
       (effects (font (size 1.27 1.27)) (justify left top))
     )
@@
     )
   )
-  (sheet (at 127.508 50.8) (size 56.134 18.542) (fields_autoplaced)
+  (sheet (at 106.68 40.64) (size 55.88 17.78) (fields_autoplaced)
     (stroke (width 0.1524) (type solid))
     (fill (color 0 0 0 0.0000))
-    (property "Sheetname" "Power" (at 127.508 50.0884 0)
+    (property "Sheetname" "Power" (at 106.68 39.9284 0)
       (effects (font (size 1.27 1.27)) (justify left bottom))
     )
-    (property "Sheetfile" "Power.kicad_sch" (at 127.508 69.9266 0)
+    (property "Sheetfile" "Power.kicad_sch" (at 106.68 59.7666 0)
       (effects (font (size 1.27 1.27)) (justify left top))
     )
@@
     )
   )
-  (sheet (at 86.36 129.54) (size 35.56 17.78) (fields_autoplaced)
+  (sheet (at 66.04 119.38) (size 35.56 17.78) (fields_autoplaced)
     (stroke (width 0.1524) (type solid))
     (fill (color 0 0 0 0.0000))
-    (property "Sheetname" "IMU" (at 86.36 128.8284 0)
+    (property "Sheetname" "IMU" (at 66.04 118.6684 0)
       (effects (font (size 1.27 1.27)) (justify left bottom))
     )
-    (property "Sheetfile" "imu.kicad_sch" (at 86.36 147.9046 0)
+    (property "Sheetfile" "imu.kicad_sch" (at 66.04 137.7446 0)
       (effects (font (size 1.27 1.27)) (justify left top))
     )
@@
     )
   )
-  (sheet (at 69.85 82.042) (size 35.306 25.908) (fields_autoplaced)
+  (sheet (at 50.8 71.12) (size 33.02 27.94)
     (stroke (width 0.1524) (type solid))
     (fill (color 0 0 0 0.0000))
-    (property "Sheetname" "Distance_sensors" (at 69.85 81.3304 0)
+    (property "Sheetname" "Distance_sensors" (at 50.8 70.4084 0)
       (effects (font (size 1.27 1.27)) (justify left bottom))
     )
-    (property "Sheetfile" "DistanceSensors.kicad_sch" (at 69.85 108.5346 0)
+    (property "Sheetfile" "DistanceSensors.kicad_sch" (at 50.8 101.6 0)
       (effects (font (size 1.27 1.27)) (justify left top))
     )
@@
     )
   )
-  (sheet (at 133.35 81.788) (size 35.179 57.15) (fields_autoplaced)
+  (sheet (at 114.3 71.12) (size 33.02 58.42)
     (stroke (width 0.1524) (type solid))
     (fill (color 0 0 0 0.0000))
-    (property "Sheetname" "Microcontroller" (at 133.35 81.0764 0)
+    (property "Sheetname" "Microcontroller" (at 114.3 70.4084 0)
       (effects (font (size 1.27 1.27)) (justify left bottom))
     )
-    (property "Sheetfile" "Microcontroller.kicad_sch" (at 133.35 139.5226 0)
+    (property "Sheetfile" "Microcontroller.kicad_sch" (at 114.3 129.54 0)
       (effects (font (size 1.27 1.27)) (justify left top))
     )
