File: DistanceSensors.kicad_sch (KiCad schematic)
At the start: 25 parts, among them IC401 ULN2003ADR, Q401 Q_Photo_NPN, Q402 Q_Photo_NPN, Q403 Q_Photo_NPN, Q404 Q_Photo_NPN, Q405 Q_Photo_NPN, Q406 Q_Photo_NPN

Commit message: Dodaje wszystko nie chce mi sie z tym bawic
Parts:
- added C403 (x6): 100n, Capacitor_SMD:C_0603_1608Metric, symbol Device:C_Small
- D401, D402, D403, D404, D405: footprint (none) -> LED_SMD:LED_0603_1608Metric
- D406: value LED -> SFH 4550; footprint (none) -> LED_SMD:LED_0603_1608Metric
- Q401: value Q_Photo_NPN -> SFH 300 FA-3/4; footprint (none) -> Connector_PinHeader_2.54mm:PinHeader_1x02_P2.54mm_Vertical
- Q402, Q403, Q404, Q405, Q406: footprint (none) -> Connector_PinHeader_2.54mm:PinHeader_1x02_P2.54mm_Vertical
- R208: footprint (none) -> Resistor_SMD:R_0603_1608Metric
Connections:
- net +5V: no longer Q401.1 (C), Q402.1 (C), Q403.1 (C), Q404.1 (C), Q405.1 (C), Q406.1 (C)
- net GND: now also C403.2, C403.2, C403.2, C403.2, C403.2, C403.2
- net Emitter_5: now reaches D402.1 (K), IC401.12 (5C)
- net at D402.2 (A), R208.2: now also C403.1
- net at D401.2 (A), R208.2: now also C403.1
- net at D406.2 (A), R208.2: now also C403.1
- net at D403.2 (A), R208.2: now also C403.1
- net Emitter_6: now reaches D401.1 (K), IC401.11 (6C)
- net Emitter_4: now reaches D403.1 (K), IC401.13 (4C)
- net Emitter_3: now reaches D404.1 (K), IC401.14 (3C)
- net Emitter_2: now reaches D405.1 (K), IC401.15 (2C)
- net Emitter_1: now reaches D406.1 (K), IC401.16 (1C)
- net at D405.2 (A), R208.2: now also C403.1
- net at D404.2 (A), R208.2: now also C403.1
- new net +3V3: Q401.1 (C), Q402.1 (C), Q403.1 (C), Q404.1 (C), Q405.1 (C), Q406.1 (C)
Other:
- note added: "Drawn by: Adam Iwachów"
- note added: "Wave length 860nm"
- note added: "Wave length 880nm"
- note added: "[5] IR RECEIVERS & EMITTERS"
- note removed: "-Nazwać lepiej wyprowadzenia, poprawadzić do uc"
- note removed: "TO DO"
- note removed: "[5] IR RECEIVERS & TRANSMITERS"
- moved on the sheet: D401, D402, D403, D404, D405, D406

Commit message: drobne zmiany
Parts:
- D501: renamed from D406; footprint LED_SMD:LED_0603_1608Metric -> Connector_PinHeader_2.54mm:PinHeader_1x02_P2.54mm_Vertical
- D502: renamed from D405; footprint LED_SMD:LED_0603_1608Metric -> Connector_PinHeader_2.54mm:PinHeader_1x02_P2.54mm_Vertical
- D503: renamed from D404; footprint LED_SMD:LED_0603_1608Metric -> Connector_PinHeader_2.54mm:PinHeader_1x02_P2.54mm_Vertical
- D504: renamed from D403; footprint LED_SMD:LED_0603_1608Metric -> Connector_PinHeader_2.54mm:PinHeader_1x02_P2.54mm_Vertical
- D505: renamed from D402; footprint LED_SMD:LED_0603_1608Metric -> Connector_PinHeader_2.54mm:PinHeader_1x02_P2.54mm_Vertical
- D506: renamed from D401; footprint LED_SMD:LED_0603_1608Metric -> Connector_PinHeader_2.54mm:PinHeader_1x02_P2.54mm_Vertical
- renumbered IC401 to IC501, Q401 to Q501, Q402 to Q502, Q403 to Q503, Q404 to Q504, Q405 to Q505, Q406 to Q506
