File: Microcontroller.kicad_sch (KiCad schematic)
At the start: 42 parts, among them J301 Conn_02x05_Counter_Clockwise, SW204 USER, SW302 USER, SW303 NRST, SW304 USER, SW601 SW_SPDT, U302 STM32F405RGT6, Y302 16MHz|9p|10ppm

Commit message: drobne zmiany
Parts:
- added C321: 100n, Capacitor_SMD:C_0603_1608Metric, symbol Device:C_Small
- added C322: 10u, Capacitor_SMD:C_0603_1608Metric, symbol Device:C_Small
- added D305, D306, D307: LED_WHITE, Diode_SMD:D_0603_1608Metric, symbol Device:LED
- added IC301: ESP32-S3-WROOM-1-N4, SamacSys_Parts:ESP32S3WROOM1N4, symbol SamacSys_Parts:ESP32-S3-WROOM-1-N4
- added R309, R310, R318: 1k, Resistor_SMD:R_0603_1608Metric, symbol Device:R_Small
- added R312, R313, R314, R315, R316: 100, Resistor_SMD:R_0603_1608Metric, symbol Device:R_Small
- added R317: 0, Resistor_SMD:R_0603_1608Metric, symbol Device:R_Small
- R307: renamed from R305; value R_Small -> 1k
- R308: renamed from R306; value R_Small -> 1k
- renumbered C315 to C301, C313 to C302, C305 to C303, C314 to C304, C316 to C305, C317 to C306, C306 to C307, C319 to C308, C320 to C309, C322 to C310, C321 to C311, C324 to C312, C323 to C313, C325 to C314, C326 to C315, C304 to C316, C302 to C317, C303 to C318, C318 to C319, C206 to C320, D304 to D303, FB302 to FB301, R309 to R301, R310 to R302, R307 to R303, R302 to R304, R304 to R305, R303 to R306, R208 to R311, SW303 to SW301, SW302 to SW303, SW204 to SW305, U302 to U301, Y302 to Y301
Connections:
- net +3.3V: now also C321.1, C322.1, IC301.2 (3V3)
- net ESP_USB_DN: now also IC301.13 (IO19); no longer C320.1, R311.1, SW305.1 (A), SW305.2 (A)
- net ESP_USB_DP: now also IC301.14 (IO20)
- net GND: now also C321.2, C322.2, D305.1 (K), D306.1 (K), D307.1 (K), IC301.1 (GND_1), IC301.40 (GND_2), IC301.41 (GND_3), IC301.42 (GND_4), IC301.43 (GND_5), IC301.44 (GND_6), IC301.45 (GND_7), IC301.46 (GND_8), IC301.47 (GND_9), IC301.48 (GND_10), IC301.49 (GND_11)
- net SPI1_CS_ESP: now also R315.1
- net SPI1_MISO_ESP: now also R316.1
- net SPI1_MOSI_ESP: now also R317.1
- net SPI1_SCK: now also R314.1
- net UART4_RX renamed UART4_RX_OTA
- net UART4_RX_OTA: now also R313.1
- net UART4_TX renamed UART4_TX_OTA
- net UART4_TX_OTA: now also R312.1
- new net: IC301.24 (IO47), R316.2
- new net: IC301.18 (IO10), R312.2
- new net: IC301.19 (IO11), R313.2
- new net: IC301.22 (IO14), R315.2
- new net: IC301.23 (IO21), R314.2
- new net: IC301.25 (IO48), R317.2
- new net: C320.1, IC301.3 (EN), R311.1, SW305.1 (A), SW305.2 (A)
- new net USER_LD2_A_esp: D306.2 (A), R310.2
- new net USER_LD2_esp: IC301.33 (IO40), IC301.34 (IO41), R309.1, R310.1
- new net USER_LD3_A_esp: D307.2 (A), R318.2
- new net USER_LD3_esp: IC301.35 (IO42), R318.1
- new net USER_LD_A_esp: D305.2 (A), R309.2
- no-connect marks 17 -> 42
Other:
- moved on the sheet: C301, C302, C303, C304, C305, C306, C307, C308, C309, C310, C311, C312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
