File: Motors.kicad_sch (KiCad schematic)
At the start: 0 parts

Commit message: DC driver
Parts:
- added C301: C_Small, symbol Device:C_Small
- added J301, J302: Conn_01x02, symbol Connector_Generic:Conn_01x02
- added NT301: ~, symbol Device:NetTie_2
- added R301: R_Small, symbol Device:R_Small
- added U301: TB6612FNG, Package_SO:SSOP-24_5.3x8.2mm_P0.65mm, symbol Driver_Motor:TB6612FNG
Connections:
- new net: J302.1 (Pin_1), U301.11 (BO1), U301.12 (BO1)
- new net: J302.2 (Pin_2), U301.7 (BO2), U301.8 (BO2)
- new net: J301.1 (Pin_1), U301.1 (AO1), U301.2 (AO1)
- new net: J301.2 (Pin_2), U301.5 (AO2), U301.6 (AO2)
- new net: C301.1, R301.2, U301.19 (STBY)
- new net +3.3V: R301.1, U301.20 (VCC)
- new net +6V: U301.13 (VM2), U301.14 (VM3), U301.24 (VM1)
- new net GND: C301.2, NT301.1, U301.18 (GND)
- new net GNDPWR: NT301.2, U301.10 (PGND2), U301.3 (PGND1), U301.4 (PGND1), U301.9 (PGND2)
- new net MotorL_BIN1: U301.17 (BIN1)
- new net MotorL_BIN2: U301.16 (BIN2)
- new net MotorL_PWM: U301.15 (PWMB)
- new net MotorR_AIN1: U301.21 (AIN1)
- new net MotorR_AIN2: U301.22 (AIN2)
- new net MotorR_PWM: U301.23 (PWMA)
Other:
- note added: "Connect ground with power ground in one place"

Commit message: Prawie skończone
Connections:
- net +6V renamed +BATT
Other:
- note added: "-Dodać enkodery"
- note added: "TO DO"
- note added: "[4] MOTORS"
- moved on the sheet: C301, J301, J302, NT301, R301, U301

Commit message: Dodaje wszystko nie chce mi sie z tym bawic
Parts:
- removed J301, J302: Conn_01x02, symbol Connector_Generic:Conn_01x02
- removed NT301: ~, symbol Device:NetTie_2
- added C201: 10u, Capacitor_Tantalum_SMD:CP_EIA-3216-10_Kemet-I_Pad1.58x1.35mm_HandSolder, symbol Device:C_Polarized_Small
- added C401, C402, C403: 100n, Capacitor_SMD:C_0603_1608Metric, symbol Device:C_Small
- added J401, J402: Conn_01x06, Connector_PinHeader_2.54mm:PinHeader_1x06_P2.54mm_Vertical, symbol Connector_Generic:Conn_01x06
- C301: value C_Small -> 100n; footprint (none) -> Capacitor_SMD:C_0603_1608Metric
- R301: value R_Small -> 10k; footprint (none) -> Resistor_SMD:R_0603_1608Metric
Connections:
- net GNDPWR is gone; now on net GND: U301.10 (PGND2), U301.3 (PGND1), U301.4 (PGND1), U301.9 (PGND2)
- net +3.3V: now also C201.1, C401.1, C402.1, C403.1, J401.4 (Pin_1), J402.4 (Pin_1)
- net GND: now also C201.2, C401.2, C402.2, C403.2, J401.1 (Pin_6), J402.1 (Pin_6)
- net BO1: now reaches U301.11 (BO1), U301.12 (BO1)
- net BO1: now also J402.6 (Pin_3)
- net BO2: now reaches U301.7 (BO2), U301.8 (BO2)
- net BO2: now also J402.5 (Pin_5)
- net AO1: now reaches U301.1 (AO1), U301.2 (AO1)
- net AO1: now also J401.6 (Pin_3)
- net AO2: now reaches U301.5 (AO2), U301.6 (AO2)
- net AO2: now also J401.5 (Pin_5)
- new net TIM_ENCODER_A1: J401.3 (Pin_4)
- new net TIM_ENCODER_A2: J402.3 (Pin_4)
- new net TIM_ENCODER_B1: J401.2 (Pin_2)
- new net TIM_ENCODER_B2: J402.2 (Pin_2)
Other:
- note added: "Drawn by: Adam Iwachów"
- note added: "Motor header & Encoders"
- note added: "TRZEBA DODAĆ UCHWYTY TO MOCOWANIA SILNIKÓW!"
- note added: "optionally"
- note added: "per encoder"
- note removed: "-Dodać enkodery"
- note removed: "Connect ground with power ground in one place"
- note removed: "TO DO"
- moved on the sheet: C301, R301, U301

Commit message: footprinty
Other:
- note added: "TRZEBA DODAĆ UCHWYTY DO MOCOWANIA SILNIKÓW!"
- note removed: "TRZEBA DODAĆ UCHWYTY TO MOCOWANIA SILNIKÓW!"
Changed lines of the file:
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@@
     (effects (font (size 1.27 1.27) bold) (justify left bottom))
   )
-  (text "TRZEBA DODAĆ UCHWYTY TO MOCOWANIA SILNIKÓW!" (at 114.3 149.86 0)
+  (text "TRZEBA DODAĆ UCHWYTY DO MOCOWANIA SILNIKÓW!" (at 114.3 149.86 0)
     (effects (font (size 1.27 1.27) (thickness 0.254) bold (color 255 18 16 1)) (justify left bottom))
   )

Commit message: drobne zmiany
Parts:
- renumbered C301 to C401, C401 to C404, C402 to C405, R301 to R401, U301 to U401
