File: imu.kicad_sch (KiCad schematic)
At the start: 3 parts, among them IC9 BMI088

Commit message: Dodaje wszystko nie chce mi sie z tym bawic
Parts:
- C410, C411: footprint Capacitor_SMD:C_0402_1005Metric -> Capacitor_SMD:C_0603_1608Metric
Other:
- note added: "Drawn by: Adam Iwachów"
- note removed: "- Jakie IMU? BMI088 testowane sprawdza się dobrze"
- note removed: "TO DO"
Changed lines of the file:
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@@
     (fill (type none))
-  )
-  (rectangle (start 147.32 30.48) (end 185.42 66.04)
-    (stroke (width 0.5) (type default) (color 255 14 41 1))
-    (fill (type none))
-  )
-  (text "- Jakie IMU? \nBMI088 testowane sprawdza\nsię dobrze "
-    (at 148.8477 43.5508 0)
-    (effects (font (size 1.5 1.5)) (justify left bottom))
   )
   (text "I2C addr. \nAcc:  0011000 << 1\nGyro: 1101000 << 1" (at 53.34 40.64 0)
@@
   )
   (text "BMI088 komunikuje się \nprzez I2C lub SPI, \nwada spi w tym sensorze jest taka, \nże potrzebne są dwa piny cs \njeden dla akcelerometru,\n drugi dla żyroskopu "
-    (at 152.4 93.98 0)
+    (at 157.48 96.52 0)
     (effects (font (size 1.27 1.27)) (justify left bottom))
   )
-  (text "TO DO " (at 147.9181 35.8038 0)
-    (effects (font (size 3 3) (thickness 0.6) bold) (justify left bottom))
-  )
-  (text "BMI088\n" (at 22.86 99.06 0)
+  (text "Drawn by: Adam Iwachów " (at 93.98 111.76 0)
+    (effects (font (size 2 2)) (justify left bottom))
+  )
+  (text "BMI088\n" (at 20.32 99.06 0)
     (effects (font (size 2 2) (thickness 0.6) bold) (justify left bottom))
   )
-  (text "*Note" (at 151.384 81.28 0)
+  (text "*Note" (at 156.464 83.82 0)
     (effects (font (size 1.27 1.27) (thickness 0.254) bold) (justify left bottom))
   )
@@
       (effects (font (size 1.27 1.27)) (justify left))
     )
-    (property "Footprint" "Capacitor_SMD:C_0402_1005Metric" (at 120.142 59.182 0)
+    (property "Footprint" "Capacitor_SMD:C_0603_1608Metric" (at 120.142 59.182 0)
       (effects (font (size 1.27 1.27)) hide)
     )
@@
       (effects (font (size 1.27 1.27)) (justify left))
     )
-    (property "Footprint" "Capacitor_SMD:C_0402_1005Metric" (at 129.667 59.182 0)
-      (effects (font (size 1.27 1.27)) hide)
-    )
+    (property "Footprint" "Capacitor_SMD:C_0603_1608Metric" (at 129.667 59.182 0)
+      (effects (font (size 1.27 1.27)) hide)
+    )
