File: adapter_STM32/adapter_STM32.kicad_sch (KiCad schematic)
At the start: 22 parts, among them J1 Conn_02x06_Top_Bottom_Mountin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, J2 Conn_02x06_Top_Bottom_Mountin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, J3 Conn_02x06_Top_Bottom_Mountin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, J4 Conn_02x06_Top_Bottom_Mountin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, U1 STM32F071CBTx, Y1 8MHz

Commit message: Dodaje wszystko nie chce mi sie z tym bawic
Parts:
- removed C1, C12, C13, C14, C15, C16, C2, C3, C4, C5, C6, C7, C8, C9: 100nF, Capacitor_SMD:C_0603_1608Metric, symbol Device:C
- removed C10, C11: 33pF, Capacitor_SMD:C_0603_1608Metric, symbol Device:C
- removed U1: STM32F071CBTx, Package_QFP:LQFP-48_7x7mm_P0.5mm, symbol MCU_ST_STM32F0:STM32F071CBTx
- added C101, C102, C103, C104, C110: 100n, symbol Device:C_Small
- added C105: 4u7, symbol Device:C_Small
- added C106: 10n, symbol Device:C_Small
- added C107: 1u, symbol Device:C_Small
- added C108, C109: 33p, symbol Device:C_Small
- added FB101: FerriteBead_Small, symbol Device:FerriteBead_Small
- added IC101: STM32F302CBT6, QFP50P900X900X160-48N, symbol SamacSys_Parts:STM32F302CBT6
- added JP101: Jumper_2_Open, symbol Jumper:Jumper_2_Open
- added R101: 10k, symbol Device:R_Small
- added R102: 0, symbol Device:R_Small
- added R103: 100, symbol Device:R_Small
- added SW101: SW_MEC_5G, symbol Switch:SW_MEC_5G
Connections:
- net BOOT0: now also IC101.44 (BOOT0), R101.1; no longer J3.5 (Pin_5)
- net NRST: now also IC101.7 (NRST), R103.2; no longer J1.6 (Pin_6)
- net PA0: now also IC101.10 (PA0); no longer J1.3 (Pin_3)
- net PA1: now also IC101.11 (PA1); no longer J1.2 (Pin_2)
- net PA10: now also IC101.31 (PA10); no longer J4.6 (Pin_6)
- net PA11: now also IC101.32 (PA11); no longer J4.5 (Pin_5)
- net PA12: now also IC101.33 (PA12); no longer J4.4 (Pin_4)
- net PA15: now also IC101.38 (PA15); no longer J3.12 (Pin_12)
- net PA2: now also IC101.12 (PA2); no longer J1.1 (Pin_1)
- net PA3: now also IC101.13 (PA3); no longer J2.11 (Pin_11)
- net PA4: now also IC101.14 (PA4); no longer J2.12 (Pin_12)
- net PA5: now also IC101.15 (PA5); no longer J2.9 (Pin_9)
- net PA6: now also IC101.16 (PA6); no longer J2.10 (Pin_10)
- net PA7: now also IC101.17 (PA7); no longer J2.7 (Pin_7)
- net PA8: now also IC101.29 (PA8); no longer J4.7 (Pin_7)
- net PA9: now also IC101.30 (PA9); no longer J4.8 (Pin_8)
- net PB0: now also IC101.18 (PB0); no longer J2.8 (Pin_8)
- net PB1: now also IC101.19 (PB1); no longer J2.6 (Pin_6)
- net PB10: now also IC101.22 (PB11); no longer J2.4 (Pin_4)
- net PB11: now also IC101.21 (PB10); no longer J2.3 (Pin_3)
- net PB12: now also IC101.25 (PB12); no longer J4.11 (Pin_11)
- net PB13: now also IC101.26 (PB13); no longer J4.12 (Pin_12)
- net PB14: now also IC101.27 (PB14); no longer J4.9 (Pin_9)
- net PB15: now also IC101.28 (PB15); no longer J4.10 (Pin_10)
- net PB2: now also IC101.20 (PB2); no longer J2.5 (Pin_5)
- net PB3: now also IC101.39 (PB3); no longer J3.9 (Pin_9)
- net PB4: now also IC101.40 (PB4); no longer J3.10 (Pin_10)
- net PB5: now also IC101.41 (PB5); no longer J3.7 (Pin_7)
- net PB6: now also IC101.42 (PB6); no longer J3.8 (Pin_8)
- net PB7: now also IC101.43 (PB7); no longer J3.6 (Pin_6)
- net PB8: now also IC101.45 (PB8); no longer J3.4 (Pin_4)
- net PB9: now also IC101.46 (PB9); no longer J3.3 (Pin_3)
- net PC13: now also IC101.2 (PC13); no longer J1.12 (Pin_12)
- net PC14: now also IC101.3 (PC14/OSC32_IN); no longer J1.9 (Pin_9)
- net PC15: now also IC101.4 (PC15/OSC32_OUT); no longer J1.10 (Pin_10)
- net VDDA: now also C107.1, FB101.1, JP101.1 (A); no longer J1.4 (Pin_4)
- net at Y1.1: now also C108.1, R102.1
- net at Y1.2: now also C109.1, IC101.6 (PF1/OSC_OUT)
- net PA13: no longer names the net of J4.3 (Pin_3)
- net PA14: no longer names the net of J3.11 (Pin_11)
- net VBAT: no longer names the net of J1.11 (Pin_11)
- net VDD: no longer names the net of J3.1 (Pin_1)
- net VDD: no longer J2.1 (Pin_1)
- net VDDIO2: no longer names the net of J4.1 (Pin_1)
- removed net VSS: J1.7 (Pin_7), J1.8 (Pin_8), J2.2 (Pin_2), J3.2 (Pin_2), J4.2 (Pin_2)
- net VSSA: no longer names the net of J1.5 (Pin_5)
- new net: C110.1, R103.1, SW101.3 (B), SW101.4 (B)
- new net: C106.1, FB101.2, IC101.9 (VDDA), JP101.2 (B)
- new net: IC101.5 (PF0/OSC_IN), R102.2
- new net +3V3: C101.1, C102.1, C103.1, C104.1, C105.1, IC101.1 (VBAT), IC101.24 (VDD_1), IC101.36 (VDD_2), IC101.48 (VDD_3)
- new net +BATT: J1.12 (Pin_12)
- new net GND: C101.2, C102.2, C103.2, C104.2, C105.2, C106.2, C107.2, C108.2, C109.2, C110.2, IC101.23 (VSS_1), IC101.35 (VSS_2), IC101.47 (VSS_3), IC101.8 (VSSA/VREF-), R101.2, SW101.1 (A), SW101.2 (A)
- new net SWCLK: IC101.37 (PA14)
- new net SWDIO: IC101.34 (PA13)
Other:
- moved on the sheet: Y1
