File: adapter_STM32/adapter_STM32.kicad_pcb (KiCad board)
At the start: 2 copper layers, 30.5 x 30.5 mm, 22 parts, among them J1 Conn_02x06_Top_Bottom_Mountin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, J2 Conn_02x06_Top_Bottom_Mountin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, J3 Conn_02x06_Top_Bottom_Mountin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, J4 Conn_02x06_Top_Bottom_Mountin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, U1 STM32F071CBTx, Y1 8MHz

Commit message: druga wersja płytki stm32 do recenzji
Parts:
- removed C1, C12, C13, C14, C15, C16, C2, C5: 100nF, Capacitor_SMD:C_0603_1608Metric
- added C17: 1uF, Capacitor_THT:CP_Radial_D5.0mm_P2.00mm, B.Cu at (85.4, 67.4)
- added ZWORKA_VBAT1: SAME PADY DO ZWARCIA, Resistor_SMD:R_0201_0603Metric, F.Cu at (87.9, 48.8)
- added ZWORKA_VDDA1: SAME PADY DO ZWARCIA, Resistor_SMD:R_0201_0603Metric, B.Cu at (90.1, 65.0)
- added ZWORKA_VSSA1: SAME PADY DO ZWARCIA, Resistor_SMD:R_0201_0603Metric, B.Cu at (90.1, 66.3)
- C10, C11: value 33pF -> 20pF
- C3: value 100nF -> 4,7uF; footprint Capacitor_SMD:C_0603_1608Metric -> Capacitor_THT:CP_Radial_D5.0mm_P2.00mm
- C4, C6: footprint Capacitor_SMD:C_0603_1608Metric -> Capacitor_SMD:C_0402_1005Metric
- C7: footprint Capacitor_SMD:C_0603_1608Metric -> Capacitor_SMD:C_0402_1005Metric; moved to F.Cu
- C8, C9: value 100nF -> 10nF; footprint Capacitor_SMD:C_0603_1608Metric -> Capacitor_SMD:C_0402_1005Metric
- J1, J2, J3, J4: value Conn_02x06_Top_Bottom_MountingPin -> Conn_02x06_Odd_Even_MountingPin
- U1: value STM32F071CBTx -> STM32F302CBTx
- Y1: value 8MHz -> 8-32MHz
- moved C9 20.2 mm to (89.8, 59.6), turned to 135 degrees
- moved C3 16.8 mm to (107.7, 67.3)
- moved C4 16.2 mm to (100.6, 62.6), turned to 0 degrees
- moved C8 13.1 mm to (88.9, 61.0), turned to 180 degrees
- moved C7 12.2 mm to (100.7, 54.3), turned to 90 degrees
- moved C6 9.89 mm to (92.4, 54.2), turned to 180 degrees
- moved J4 1.27 mm to (109.2, 50.8)
- moved J1 1.27 mm to (83.8, 63.5)
Connections:
- C3 pad 1: VSS -> VDD
- C3 pad 2: VDDA -> VSS
- C4 pad 1: VSS -> VDD
- C4 pad 2: VDDIO2 -> VSS
- C6 pad 1: VSS -> VDD
- C6 pad 2: VDD -> VSS
- C7 pad 1: VSS -> VDD
- C7 pad 2: VDDA -> VSS
- C8 pad 1: VSS -> VDDA
- C8 pad 2: VDD -> VSSA
- C9 pad 1: VSS -> VDDA
- C9 pad 2: VDDIO2 -> VSSA
- J2 pad 1: VDD -> VSS
- J2 pad 2: VSS -> VDD
- J3 pad 1: VDD -> VSS
- J3 pad 2: VSS -> VDD
- J4 pad 1: VDDIO2 -> VSS
- J4 pad 2: VSS -> VDD
- U1 pad 36: VDDIO2 -> VDD
Routing:
- net VSSA: track 9.80 -> 28.2 mm
- net VDD: track 30.5 -> 47.1 mm
- net VDDIO2: track 14.9 -> 0.00 mm
- net VSS: track 0.00 -> 6.64 mm, vias 3 -> 4
- net VDDA: track 23.8 -> 18.3 mm
- net PB15: track 8.43 -> 11.5 mm
- net PA2: track 13.7 -> 11.1 mm
- net PA0: track 13.2 -> 10.9 mm
- net PB14: track 11.2 -> 13.6 mm
- net PB13: track 8.44 -> 9.82 mm
- net PC13: track 8.44 -> 9.53 mm
- net NRST: track 7.14 -> 6.10 mm
- net VBAT: track 14.7 -> 13.7 mm
- net PA1: track 8.44 -> 7.69 mm
- net PB12: track 11.9 -> 12.6 mm
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- added copper zone on F.Cu, net VSSA
Other:
- board text added: "100nF"
- board text added: "10nF"
- board text added: "20pF"
- board text added: "Standardowy adapter STM32 LQFP48 projekt: Adam Wąs KNR KoNaR / Projekt 02"
- board text added: "zworka_VBAT ----->"
- board text added: "zworka_VDDA"
- board text added: "zworka_VSSA"
- board text removed: "Standardowy adapter STM32 projekt: Adam Wąs KNR KoNaR / Projekt 02"
- board text removed: "Wartości C0603: 33pF - przy krysztale 100nF - pozostałe"

Commit message: zapomniałem kilku ścieżek, teraz jest całość
Parts:
- moved C17 0.07 mm to (85.3, 67.3)
Routing:
- net VDD: track 47.1 -> 49.7 mm
Changed lines of the file:
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@@
   )
   (footprint "Capacitor_THT:CP_Radial_D5.0mm_P2.00mm" (layer "B.Cu")
-    (at 85.3948 67.3608 -90)
+    (at 85.344 67.31 -90)
     (descr "CP, Radial series, Radial, pin pitch=2.00mm, , diameter=5mm, Electrolytic Capacitor")
     (tags "CP Radial series Radial pin pitch 2.00mm  diameter 5mm Electrolytic Capacitor")
@@
         (effects (font (size 1 1) (thickness 0.15)) (justify mirror))
     )
-    (fp_text value "1uF" (at 4.4704 -0.6096 180) (layer "B.SilkS")
+    (fp_text value "1uF" (at 0 3.302 -90) (layer "B.SilkS")
         (effects (font (size 1 1) (thickness 0.15)) (justify mirror))
     )
@@
     (property "ki_keywords" "connector")
     (attr through_hole)
-    (fp_text reference "J4" (at 1.27 -14.986) (layer "B.SilkS")
+    (fp_text reference "J4" (at -1.27 -15.24) (layer "B.SilkS")
         (effects (font (size 1 1) (thickness 0.15)) (justify mirror))
     )
@@
         (effects (font (size 1 1) (thickness 0.15)) (justify mirror))
     )
-    (fp_text value "4,7uF" (at 4.5212 1.4732) (layer "B.SilkS")
+    (fp_text value "4,7uF" (at 4.064 1.524 -30) (layer "B.SilkS")
         (effects (font (size 1 1) (thickness 0.15)) (justify mirror))
     )
@@
     (property "ki_keywords" "connector")
     (attr through_hole)
-    (fp_text reference "J3" (at 1.27 -15.24) (layer "B.SilkS")
+    (fp_text reference "J3" (at -1.27 -15.24) (layer "B.SilkS")
         (effects (font (size 1 1) (thickness 0.15)) (justify mirror))
     )
@@
     (property "ki_keywords" "connector")
     (attr through_hole)
-    (fp_text reference "J2" (at 1.27 -15.24) (layer "B.SilkS")
+    (fp_text reference "J2" (at -1.27 -15.24) (layer "B.SilkS")
         (effects (font (size 1 1) (thickness 0.15)) (justify mirror))
     )
@@
     (property "ki_keywords" "connector")
     (attr through_hole)
-    (fp_text reference "J1" (at 1.27 -14.986) (layer "B.SilkS")
+    (fp_text reference "J1" (at -1.27 -14.986) (layer "B.SilkS")
         (effects (font (size 1 1) (thickness 0.15)) (justify mirror))
     )
@@
   (segment (start 93.472 52.872) (end 92.202 52.872) (width 0.3) (layer "F.Cu") (net 22))
   (segment (start 100.838 63.968) (end 102.87 66) (width 0.3) (layer "F.Cu") (net 22))
+  (segment (start 92.9132 54.1528) (end 93.6752 54.1528) (width 0.5) (layer "F.Cu") (net 22))
   (segment (start 105.3675 50.8) (end 106.68 50.8) (width 0.3) (layer "F.Cu") (net 22))
   (segment (start 93.77 53.17) (end 93.472 52.872) (width 0.3) (layer "F.Cu") (net 22))
+  (segment (start 100.7364 54.7852) (end 100.7364 55.6124) (width 0.4) (layer "F.Cu") (net 22))
   (segment (start 100.644 55.666) (end 101.7715 55.666) (width 0.3) (layer "F.Cu") (net 22))
   (segment (start 102.0695 55.368) (end 102.0695 54.098) (width 0.3) (layer "F.Cu") (net 22))
   (segment (start 102.87 66) (end 102.87 68.58) (width 0.3) (layer "F.Cu") (net 22))
   (segment (start 99.568 63.968) (end 100.838 63.968) (width 0.3) (layer "F.Cu") (net 22))
+  (segment (start 100.7364 55.6124) (end 100.6856 55.6632) (width 0.25) (layer "F.Cu") (net 22))
   (segment (start 107.696 67.31) (end 104.14 67.31) (width 1) (layer "F.Cu") (net 22))
   (segment (start 90.17 50.84) (end 90.17 48.26) (width 0.3) (layer "F.Cu") (net 22))
@@
   (segment (start 99.27 62.5425) (end 99.27 63.67) (width 0.3) (layer "F.Cu") (net 22))
   (segment (start 101.7715 55.666) (end 102.0695 55.368) (width 0.3) (layer "F.Cu") (net 22))
+  (segment (start 100.104 62.6364) (end 99.3338 62.6364) (width 0.5) (layer "F.Cu") (net 22))
+  (segment (start 93.6752 54.1528) (end 93.7731 54.2507) (width 0.25) (layer "F.Cu") (net 22))
   (segment (start 99.27 63.67) (end 99.568 63.968) (width 0.3) (layer "F.Cu") (net 22))
   (segment (start 90.17 48.26) (end 88.113 48.26) (width 0.3) (layer "F.Cu") (net 22))
+  (segment (start 99.3338 62.6364) (end 99.2731 62.5757) (width 0.25) (layer "F.Cu") (net 22))
   (segment (start 90.399 65.024) (end 99.314 65.024) (width 0.3) (layer "B.Cu") (net 22))
   (segment (start 99.314 65.024) (end 102.87 68.58) (width 0.3) (layer "B.Cu") (net 22))
@@
     (polygon
       (pts
-        (xy 90.932 58.674)
-        (xy 90.932 59.436)
-        (xy 89.662 59.436)
-        (xy 89.408 59.69)
-        (xy 89.408 60.452)
-        (xy 88.646 60.452)
-        (xy 88.646 61.468)
-        (xy 89.408 61.468)
+        (xy 91.186 58.42)
+        (xy 91.186 59.436)
+        (xy 89.916 59.436)
+        (xy 89.662 59.69)
+        (xy 89.408 60.198)
+        (xy 88.9 60.198)
+        (xy 88.9 61.214)
+        (xy 89.408 61.214)
         (xy 89.408 61.976)
-        (xy 88.646 61.976)
+        (xy 88.646 62.23)
         (xy 87.376 61.976)
-        (xy 86.868 61.722)
-        (xy 87.376 61.214)
-        (xy 87.376 60.706)
-        (xy 86.868 60.198)
-        (xy 86.868 58.928)
-        (xy 87.63 58.674)
+        (xy 86.868 61.468)
+        (xy 87.376 60.96)
+        (xy 87.376 60.452)
+        (xy 85.852 60.198)
+        (xy 85.852 58.928)
+        (xy 87.63 58.42)
       )
     )
