File: adapter_ESP32-S3/adapter_ESP32-S3.kicad_pcb (KiCad board)
At the start: 2 copper layers, 32.6 x 38.2 mm, 11 parts, among them J1 Conn_01x11_MountingPin, J2 Conn_02x09_Odd_Even_MountingP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, J3 Conn_01x11_MountingPin, J4 USB_C_Receptacle_USB2.0, U1 AP1117-33, U2 ESP32-S3-WROOM-1-N8

Commit message: poprawione esp32s3
Parts:
- C3: value 4,7Uf -> 4,7uF
- moved R2 7.62 mm to (47.2, 70.1)
- moved R1 5.59 mm to (62.0, 70.1)
Routing:
- net Net-(J4-CC1): track 2.64 -> 8.09 mm
- net Net-(J4-CC2): track 3.50 -> 7.36 mm
